File: keyboard-main/keyboard.kicad_pcb (KiCad board)
At the start: 2 copper layers, 306 x 97 mm, 141 parts, among them J1 Conn_01x30, SW1 SW_Push, SW10 SW_Push, SW11 SW_Push, SW12 SW_Push, SW13 SW_Push, SW14 SW_Push, SW15 SW_Push, SW16 SW_Push, SW17 SW_Push, SW18 SW_Push, SW19 SW_Push, SW2 SW_Push, SW20 SW_Push, SW21 SW_Push, SW22 SW_Push, SW23 SW_Push, SW24 SW_Push, SW25 SW_Push, SW26 SW_Push, SW27 SW_Push, SW28 SW_Push, SW29 SW_Push, SW3 SW_Push, SW30 SW_Push, SW31 SW_Push, SW32 SW_Push, SW33 SW_Push, SW34 SW_Push, SW35 SW_Push, SW36 SW_Push, SW37 SW_Push, SW38 SW_Push, SW39 SW_Push, SW4 SW_Push, SW40 SW_Push, SW41 SW_Push, SW42 SW_Push, SW43 SW_Push, SW44 SW_Push, SW45 SW_Push, SW46 SW_Push, SW47 SW_Push, SW48 SW_Push, SW49 SW_Push, SW5 SW_Push, SW50 SW_Push, SW51 SW_Push, SW52 SW_Push, SW53 SW_Push, SW54 SW_Push, SW55 SW_Push, SW56 SW_Push, SW57 SW_Push, SW58 SW_Push, SW59 SW_Push, SW6 SW_Push, SW60 SW_Push, SW61 SW_Push, SW62 SW_Push, SW63 SW_Push, SW64 SW_Push, SW65 SW_Push, SW66 SW_Push, SW67 SW_Push, SW68 SW_Push, SW7 SW_Push, SW8 SW_Push, SW9 SW_Push

Commit message: Move FFC connector up 8.75mm for cable clearance; vias 0.6/0.3, island cleanup
Parts:
- moved J1 8.76 mm to (192.0, 122.0)
Routing:
- net ROW0: track 499.4 -> 358.0 mm, vias 0 -> 4
- net ROW1: track 339.4 -> 408.5 mm, vias 4 -> 2
- net ROW3: track 291.2 -> 317.5 mm, vias 10 -> 4
- net ROW4: track 289.5 -> 313.3 mm
- net GND: track 43.6 -> 27.1 mm, vias 67 -> 5
- net COL13: track 182.1 -> 195.5 mm, vias 8 -> 5
- net COL12: track 166.4 -> 179.8 mm, vias 8 -> 5
- net COL11: track 145.5 -> 156.6 mm, vias 6 -> 5
- net COL6: track 139.1 -> 147.7 mm, vias 10 -> 6
- net COL9: track 104.8 -> 113.1 mm, vias 4 -> 5
- net COL4: track 172.5 -> 180.3 mm, vias 8 -> 5
- net ROW2: track 325.6 -> 318.2 mm, vias 30 -> 4
- net COL1: track 233.8 -> 241.0 mm, vias 6 -> 5
- net COL8: track 92.6 -> 99.7 mm, vias 6 -> 5
- net Net-(D39-A): track 10.1 -> 17.2 mm, vias 0 -> 2
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